File: cliente-micro/pcb_cliente_micro_acuamet/pcb_cliente_micro_acuamet.kicad_pcb (KiCad board)
At the start: 2 copper layers, 89.5 x 57.5 mm, 40 parts, among them J1 Presion, J10 5V IN, J2 Ultrasonico, J3 Valvula 1, J4 Valvula 2, J5 Relay, J6 Debug, J7 Valvula 3, J8 LCD, J9 Valvula 4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

Commit message: PCB
Parts:
- added J11: Botones, Connector_Molex:Molex_KK-254_AE-6410-05A_1x05_P2.54mm_Vertical, F.Cu at (90.9, 42.7)
- added R18: 0, Resistor_SMD:R_0805_2012Metric_Pad1.20x1.40mm_HandSolder, B.Cu at (167.3, 68.0)
- added R19: 0, Resistor_SMD:R_0805_2012Metric_Pad1.20x1.40mm_HandSolder, B.Cu at (167.3, 70.4)
- moved R5 3.91 mm to (115.1, 63.8)
- moved J10 3.68 mm to (91.1, 60.1)
- moved R13 3.68 mm to (164.3, 61.1)
- moved R12 1.40 mm to (164.3, 63.6)
- moved R11 1.27 mm to (164.3, 58.4)
- moved REF** 1.15 mm to (92.5, 36.3), turned to -90 degrees
- moved REF** 0.25 mm to (171.7, 34.9)
Connections:
- D2 pad 1: unconnected-(D2-BA-Pad1) -> Net-(D2-BA)
- D2 pad 2: unconnected-(D2-RA-Pad2) -> Net-(D2-RA)
- D2 pad 3: unconnected-(D2-GA-Pad3) -> Net-(D2-GA)
- D2 pad 4: unconnected-(D2-K-Pad4) -> Net-(D2-K)
- R11 pad 2: unconnected-(R11-Pad2) -> Net-(D2-BA)
- R12 pad 2: unconnected-(R12-Pad2) -> Net-(D2-GA)
- R13 pad 2: unconnected-(R13-Pad2) -> Net-(D2-RA)
Routing:
- net /config_pin: track 0.00 -> 86.5 mm, vias 0 -> 1
- net +3.3V: track 42.3 -> 103.1 mm, vias 0 -> 1
- net /boton_2: track 13.0 -> 45.3 mm, vias 0 -> 1
- net /boton_0: track 11.6 -> 42.5 mm, vias 0 -> 1
- net /boton_1: track 12.6 -> 40.5 mm, vias 0 -> 1
- net /flujometro_2: track 53.5 -> 35.8 mm
- net +5V: track 219.6 -> 205.3 mm
- net /valvula_4: track 69.8 -> 59.2 mm
- net /sens_presion: track 24.9 -> 32.0 mm
- net Net-(D2-K): track 0.00 -> 6.06 mm
- net Net-(D2-GA): track 0.00 -> 4.60 mm
- net Net-(D2-RA): track 0.00 -> 4.50 mm
- net /ultrasonico_trig: track 73.4 -> 77.9 mm
- net /ultrasonico_echo: track 69.9 -> 74.1 mm
- net Net-(D2-BA): track 0.00 -> 4.23 mm
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